File: femtoduino.sch (EAGLE design)
At the start: 17 parts, among them SW1 SWITCH, U1 MIC5205, U2 ATMEGA328P-AU, Y1 16MHz

Commit message: add femtoduino brd
Parts:
- LED1: value amber -> AMBER
Changed lines of the file:
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@@
 <part name="C3" library="eagle-book" deviceset="CAP_TANT" device="" value="10uF"/>
 <part name="C4" library="eagle-book" deviceset="CAP" device="_0603" value="0.1uF"/>
-<part name="LED1" library="eagle-book" deviceset="LED" device="_0603" value="amber"/>
+<part name="LED1" library="eagle-book" deviceset="LED" device="_0603" value="AMBER"/>
 <part name="U2" library="eagle-book" deviceset="ATMEGA328P" device="-AU"/>
 <part name="Y1" library="eagle-book" deviceset="CSTCE" device="" value="16MHz"/>
