File: femtoduino.brd (EAGLE design)
At the start: 30.5 x 47 mm, 17 parts, among them SW1 SWITCH, U1 MIC5205, U2 ATMEGA328P-AU, Y1 16MHz

Commit message: routing
Routing:
- net GND: track 0.00 -> 117.9 mm, vias 0 -> 2
- net RESET: track 0.00 -> 88.0 mm, vias 0 -> 1
- net VCC: track 0.00 -> 68.8 mm, vias 0 -> 3
- net D13/SCK: track 0.00 -> 42.5 mm, vias 0 -> 1
- net AREF: track 0.00 -> 33.1 mm
- net N$5: track 0.00 -> 27.1 mm, vias 0 -> 3
- net D11/MOSI: track 0.00 -> 26.0 mm
- net D12/MISO: track 0.00 -> 23.3 mm
- net VIN: track 0.00 -> 20.8 mm
- net D2: track 0.00 -> 17.2 mm
- net D1: track 0.00 -> 15.8 mm
- net A6: track 0.00 -> 15.4 mm
- net D0: track 0.00 -> 14.4 mm
- net D10: track 0.00 -> 14.4 mm
- net D3: track 0.00 -> 14.0 mm
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